File: board/board.kicad_pcb (KiCad board)
At the start: 2 copper layers, 21 x 13 mm, 1 part

Commit message: initial
Parts:
- added J1: 020_1000BASE-T_with_CT, on_edge:on_edge_2x10_device, F.Cu at (112.0, 96.0)
- added J2: 7499111121A, b038:7499111121A, F.Cu at (127.5, 100.0)
- moved LOGO1 25.0 mm to (129.4, 113.2)
Routing:
- net /connector/LED2_C: track 0.00 -> 32.8 mm
- net /connector/LED2_A: track 0.00 -> 27.0 mm
- net /connector/CT: track 0.00 -> 27.0 mm
- net /connector/A+: track 0.00 -> 25.7 mm
- net /connector/LED1_A: track 0.00 -> 22.6 mm, vias 0 -> 1
- net /connector/A-: track 0.00 -> 21.7 mm
- net /connector/LED1_C: track 0.00 -> 21.4 mm, vias 0 -> 2
- net /connector/D-: track 0.00 -> 21.2 mm, vias 0 -> 1
- net /connector/D+: track 0.00 -> 20.8 mm, vias 0 -> 1
- net /connector/GND_schield: track 0.00 -> 17.6 mm
- net /connector/B+: track 0.00 -> 9.66 mm, vias 0 -> 1
- net /connector/C-: track 0.00 -> 9.22 mm, vias 0 -> 1
- net /connector/C+: track 0.00 -> 8.38 mm
- net /connector/GND: track 0.00 -> 7.70 mm
- net /connector/B-: track 0.00 -> 7.06 mm
Other:
- board size 21 x 13 mm -> 21 x 29 mm
- copper layers 2 -> 4
- rule pad_to_mask_clearance: 0 -> 0.051
- board text added: "osf.020"
- board text added: "osf.b038.v1.0"
